Commit message: update using laserfilters

File: examples/meshes/full_example.urdf (robot description, URDF)
Before this commit: robot NIFTi, 4 links, 3 joints
Links:
- link base_link: geometry collision box size=1.8 1.8 1.8; collision box size=2.2545 1.12545 0.7515
Joints:
- joint laser_base_j: child laser_base -> laser
- joint laser_j: child laser -> laser_base; parent laser_base -> laser
